File: ArduinoRadioV3/ArduinoRadioV3.brd (EAGLE design)
At the start: 31.7 x 34 mm, 26 parts, among them IC1 ATMEGA328P-AU, IC2 LM50, IC3 SI4703-C19-GM, J1 UJC-HP-3-SMT-TR, U1 MCP73831T-2ACI/OT, Y1 ABM3B-8.000MHZ-10-1-U-T

Commit message: Update README
Parts:
- moved R2 16.3 mm to (4.45, 8.89)
- moved L1 3.03 mm to (29.0, 21.6), turned to 180 degrees
- moved C8 2.55 mm to (27.6, 23.5)
- moved U$1 2.42 mm to (17.8, 26.8)
- moved IC3 1.40 mm to (21.2, 23.7)
- moved C7 0.38 mm to (17.7, 21.2)
Routing:
- net ROUT: track 0.00 -> 9.66 mm
- net ANT: track 0.00 -> 4.70 mm
- net N$4: track 0.00 -> 4.06 mm
- net STAT: track 2.20 -> 3.08 mm
- net LOUT: track 2.04 -> 2.90 mm
- net VBAT: track 21.4 -> 22.0 mm
